File: 2. MicroMouse PCB/PCB_AIO_V1/PCB_AIO_V1.kicad_pcb (KiCad board)
At the start: 2 copper layers, 70 x 70 mm, 57 parts, among them J1 Conn_01x02_Pin, J10 Conn_01x03_Pin, J11 Conn_01x03_Pin, J12 Conn_01x03_Pin, J13 Conn_01x06_Pin, J14 Conn_01x06_Pin, J15 Conn_01x06_Pin, J16 Conn_01x06_Pin, J2 STLINK, J3 MPU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

Commit message: completed PCB_AIO_V1
Parts:
- C14, C15: moved to F.Cu
- C2: moved to B.Cu
- J1: footprint Connector_PinSocket_2.54mm:PinSocket_1x02_P2.54mm_Vertical_SMD_Pin1Left -> Connector_JST:JST_VH_B2P-VH-B_1x02_P3.96mm_Vertical
- J10, J11, J12, J9: footprint Connector_JST:JST_SH_BM03B-SRSS-TB_1x03-1MP_P1.00mm_Vertical -> Connector_JST:JST_SH_SM03B-SRSS-TB_1x03-1MP_P1.00mm_Horizontal
- J2: footprint Connector_JST:JST_SH_SM04B-SRSS-TB_1x04-1MP_P1.00mm_Horizontal -> Connector_JST:JST_SH_BM04B-SRSS-TB_1x04-1MP_P1.00mm_Vertical
- Y1: value 48MHz -> Crystal_GND24_Small; footprint Crystal:Crystal_SMD_3225-4Pin_3.2x2.5mm_HandSoldering -> Crystal:Crystal_SMD_3225-4Pin_3.2x2.5mm; moved to F.Cu
- moved Q1 27.5 mm to (173.5, 82.4)
- moved R5 25.6 mm to (172.5, 80.1), turned to 0 degrees
- moved C5 25.3 mm to (148.0, 84.7), turned to 90 degrees
- moved J12 13.6 mm to (171.6, 99.5)
- moved J9 11.7 mm to (146.2, 99.5)
- moved R3 8.94 mm to (171.1, 91.0), turned to 0 degrees
- moved C16 8.61 mm to (171.1, 85.5), turned to 0 degrees
- moved R2 8.32 mm to (143.1, 76.8), turned to 90 degrees
- moved J10 8.31 mm to (139.3, 99.5), turned to 90 degrees
- moved SW2 8.24 mm to (175.5, 92.4)
- moved SW3 8.01 mm to (175.6, 88.0)
- moved C13 7.87 mm to (171.1, 90.0), turned to 0 degrees
- moved C15 7.76 mm to (125.9, 85.7), turned to -90 degrees
- moved R4 7.63 mm to (171.1, 86.5), turned to 0 degrees
- moved C14 7.48 mm to (125.8, 94.1), turned to 90 degrees
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Connections:
- C14 pad 2: /PH0 -> /PH1
- C15 pad 2: /PH1 -> /PH0
- Q1 pad 1: +5V -> +3.3V
- U1 pad 10: Net-(U1-GND) -> GND
- U1 pad 18: Net-(U1-GND) -> GND
- U1 pad 3: Net-(U1-GND) -> GND
- U1 pad 4: Net-(U1-GND) -> GND
- U1 pad 9: Net-(U1-GND) -> GND
- U3 pad 15: /N_TOF -> /S_TOF
- U3 pad 16: /W_TOF -> /E_TOF
- U3 pad 17: /S_TOF -> /N_TOF
- U3 pad 18: /E_TOF -> /W_TOF
- U3 pad 63: /NW_SERVO -> /SW_SERVO
- U3 pad 64: /SW_SERVO -> /SE_SERVO
- U3 pad 65: /SE_SERVO -> /NW_SERVO
- U4 pad 1: /SW_M1 -> /SE_M1
- U4 pad 10: Net-(U4-GND) -> GND
- U4 pad 11: /SE_M1 -> /SW_M1
- U4 pad 12: /SE_M1 -> /SW_M1
- U4 pad 15: /SE_PWM -> /SW_PWM
- U4 pad 16: /SE_IN2 -> /SW_IN2
- U4 pad 17: /SE_IN1 -> /SW_IN1
- U4 pad 18: Net-(U4-GND) -> GND
- U4 pad 2: /SW_M1 -> /SE_M1
- U4 pad 21: /SW_IN1 -> /SE_IN1
- U4 pad 22: /SW_IN2 -> /SE_IN2
- U4 pad 23: /SW_PWM -> /SE_PWM
- U4 pad 3: Net-(U4-GND) -> GND
- U4 pad 4: Net-(U4-GND) -> GND
- U4 pad 5: /SW_M2 -> /SE_M2
- U4 pad 6: /SW_M2 -> /SE_M2
- U4 pad 7: /SE_M2 -> /SW_M2
- U4 pad 8: /SE_M2 -> /SW_M2
- U4 pad 9: Net-(U4-GND) -> GND
- Y1 pad 1: /PH0 -> /PH1
- Y1 pad 2: /PH1 -> GND
- Y1 pad 3: (no net) -> /PH0
- Y1 pad 4: (no net) -> GND
Routing:
- net GND: track 336.5 -> 3.05 mm, vias 7 -> 195
- net +5V: track 124.3 -> 4.29 mm, vias 6 -> 12
- net /NW_IN2: track 65.9 -> 23.5 mm, vias 7 -> 1
- net /NW_PWM: track 63.0 -> 21.4 mm, vias 7 -> 1
- net /IN-: track 36.7 -> 0.00 mm, vias 2 -> 0
- net /BUTTON_1: track 80.4 -> 51.1 mm, vias 2 -> 0
- net /SE_ENC_B: track 63.5 -> 36.3 mm
- net /IN+: track 25.4 -> 0.00 mm, vias 1 -> 32
- net Net-(C5-Pad2): track 28.5 -> 3.80 mm, vias 2 -> 0
- net /NE_ENC_A: track 42.3 -> 66.6 mm, vias 3 -> 1
- net /SE_M1: track 22.7 -> 0.00 mm
- net /S_TOF: track 76.0 -> 53.7 mm, vias 3 -> 1
- net /NW_M2: track 22.3 -> 0.00 mm
- net /SE_IN1: track 48.3 -> 26.3 mm
- net /NE_ENC_B: track 43.2 -> 65.0 mm
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- added copper zone on B.Cu, net +5V
- added copper zone on F.Cu, net +5V
- added copper zone on B.Cu, net /IN+
- added copper zone on F.Cu, net /IN+
- added copper zone on B.Cu, net /IN-
- added copper zone on F.Cu, net /IN-
- added copper zone on B.Cu, net /NE_M1
- added copper zone on B.Cu, net /NE_M2
- added copper zone on B.Cu, net /NW_M1
- added copper zone on B.Cu, net /NW_M2
- added copper zone on B.Cu, net /SE_M1
- added copper zone on B.Cu, net /SE_M2
- added copper zone on B.Cu, net /SW_M1
- added copper zone on B.Cu, net /SW_M2
- added copper zone on B.Cu, net GND
- added copper zone on F.Cu, net GND
Other:
- outline, holes or cut-outs redrawn
- board text added: "ESP32 DISPLAY"
- board text added: "E_TOF"
- board text added: "MPU"
- board text added: "NE_MOTOR"
- board text added: "NE_SERVO"
- board text added: "NW_MOTOR"
- board text added: "NW_SERVO"
- board text added: "N_TOF"
- board text added: "SE_MOTOR"
- board text added: "SE_SERVO"
- board text added: "ST-LINK"
- board text added: "SW_MOTOR"
- board text added: "SW_SERVO"
- board text added: "S_TOF"
- board text added: "W_TOF"

Commit message: finish PCB_AIO_V1
Parts:
- C5: moved to B.Cu
- moved C16 20.0 mm to (187.0, 97.7), turned to 90 degrees
- moved C12 17.7 mm to (185.8, 105.3)
- moved R4 17.2 mm to (186.5, 94.1)
- moved R3 16.3 mm to (186.5, 96.1)
- moved C13 16.1 mm to (187.0, 92.5), turned to -90 degrees
- moved SW1 15.7 mm to (184.3, 109.7), turned to 90 degrees
- moved J4 11.9 mm to (177.9, 101.0)
- moved SW2 11.6 mm to (184.3, 100.0), turned to 90 degrees
- moved SW3 9.01 mm to (184.3, 90.2), turned to -90 degrees
- moved BZ1 3.57 mm to (165.5, 75.8)
- moved J8 2.99 mm to (156.2, 88.0)
- moved J7 2.99 mm to (156.2, 95.6)
- moved J5 1.81 mm to (150.9, 88.0)
- moved J6 1.81 mm to (150.9, 95.6)
- moved C5 0.81 mm to (147.9, 83.8)
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Connections:
- U3 pad 5: unconnected-(U3-PE6-Pad5) -> /BUZZER
Routing:
- net /BUZZER: track 0.00 -> 63.3 mm, vias 0 -> 2
- net /BUTTON_1: track 51.1 -> 67.6 mm
- net /BUTTON_0: track 54.0 -> 68.6 mm
- net /USART1_TX: track 45.0 -> 34.1 mm, vias 2 -> 1
- net /NRST: track 90.4 -> 100.5 mm
- net /USART1_RX: track 43.3 -> 33.2 mm
- net +3.3V: track 270.2 -> 277.8 mm
- net Net-(BZ1--): track 13.2 -> 16.6 mm
- net /NE_SERVO: track 13.6 -> 10.7 mm
- net /NW_SERVO: track 6.90 -> 5.09 mm
- net /SE_SERVO: track 14.7 -> 13.0 mm
- net /NE_ENC_B: track 65.0 -> 63.8 mm
- net /NE_ENC_A: track 66.6 -> 65.4 mm
- net /S_TOF: track 53.7 -> 54.7 mm
- net /E_TOF: track 43.5 -> 42.6 mm
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Other:
- board text added: "E_SENSOR"
- board text added: "N_SENSOR"
- board text added: "S_SENSOR"
- board text added: "W_SENSOR"
- board text removed: "E_TOF"
- board text removed: "N_TOF"
- board text removed: "S_TOF"
- board text removed: "W_TOF"
