File: 2. MicroMouse PCB/PCB_AIO_V1/PCB_AIO_V1.kicad_sch (KiCad schematic)
At the start: 57 parts, among them J1 Conn_01x02_Pin, J10 Conn_01x03_Pin, J11 Conn_01x03_Pin, J12 Conn_01x03_Pin, J13 Conn_01x06_Pin, J14 Conn_01x06_Pin, J15 Conn_01x06_Pin, J16 Conn_01x06_Pin, J2 STLINK, J3 MPU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

Commit message: completed PCB_AIO_V1
Parts:
- removed Y1: 48MHz, Crystal:Crystal_SMD_3225-4Pin_3.2x2.5mm_HandSoldering, symbol Device:Crystal
- added Y1: Crystal_GND24_Small, Crystal:Crystal_SMD_3225-4Pin_3.2x2.5mm, symbol Device:Crystal_GND24_Small
- J1: footprint Connector_PinSocket_2.54mm:PinSocket_1x02_P2.54mm_Vertical_SMD_Pin1Left -> Connector_JST:JST_VH_B2P-VH-B_1x02_P3.96mm_Vertical
- J10, J11, J12, J9: footprint Connector_JST:JST_SH_BM03B-SRSS-TB_1x03-1MP_P1.00mm_Vertical -> Connector_JST:JST_SH_SM03B-SRSS-TB_1x03-1MP_P1.00mm_Horizontal
- J2: footprint Connector_JST:JST_SH_SM04B-SRSS-TB_1x04-1MP_P1.00mm_Horizontal -> Connector_JST:JST_SH_BM04B-SRSS-TB_1x04-1MP_P1.00mm_Vertical
Connections:
- net +3.3V: now also Q1.1 (E)
- net +5V: no longer Q1.1 (E)
- net E_TOF: now also U3.16 (PC1); no longer U3.18 (PC3_C)
- net GND: now also U1.10 (PGND2), U1.18 (GND), U1.3 (PGND1), U1.4 (PGND1), U1.9 (PGND2), U4.10 (PGND2), U4.18 (GND), U4.3 (PGND1), U4.4 (PGND1), U4.9 (PGND2), Y1.2, Y1.4
- net NW_SERVO: now also U3.65 (PC8); no longer U3.63 (PC6)
- net N_TOF: now also U3.17 (PC2_C); no longer U3.15 (PC0)
- net PH0: now also C15.2, Y1.3; no longer C14.2
- net PH1: now also C14.2, Y1.1; no longer C15.2
- net SE_IN1: now also U4.21 (AIN1); no longer U4.17 (BIN1)
- net SE_IN2: now also U4.22 (AIN2); no longer U4.16 (BIN2)
- net SE_M1: now also U4.1 (AO1), U4.2 (AO1); no longer U4.11 (BO1), U4.12 (BO1)
- net SE_M2: now also U4.5 (AO2), U4.6 (AO2); no longer U4.7 (BO2), U4.8 (BO2)
- net SE_PWM: now also U4.23 (PWMA); no longer U4.15 (PWMB)
- net SE_SERVO: now also U3.64 (PC7); no longer U3.65 (PC8)
- net SW_IN1: now also U4.17 (BIN1); no longer U4.21 (AIN1)
- net SW_IN2: now also U4.16 (BIN2); no longer U4.22 (AIN2)
- net SW_M1: now also U4.11 (BO1), U4.12 (BO1); no longer U4.1 (AO1), U4.2 (AO1)
- net SW_M2: now also U4.7 (BO2), U4.8 (BO2); no longer U4.5 (AO2), U4.6 (AO2)
- net SW_PWM: now also U4.15 (PWMB); no longer U4.23 (PWMA)
- net SW_SERVO: now also U3.63 (PC6); no longer U3.64 (PC7)
- net S_TOF: now also U3.15 (PC0); no longer U3.17 (PC2_C)
- net W_TOF: now also U3.18 (PC3_C); no longer U3.16 (PC1)

Commit message: finish PCB_AIO_V1
Connections:
- net BUZZER: now also U3.5 (PE6)
Changed lines of the file:
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@@
+	(wire
+		(pts
+			(xy 116.078 165.608) (xy 119.888 165.608)
+		)
+		(stroke
+			(width 0)
+			(type default)
+		)
+	)
 	(wire
 		(pts
@@
 			)
 			(justify right bottom)
+		)
+	)
+	(label "BUZZER"
+		(at 116.078 165.608 180)
+		(fields_autoplaced yes)
+		(effects
+			(font
+				(size 1.27 1.27)
+			)
+			(justify right bottom)
