File: 2. MicroMouse PCB/PCB_AIO_V2/PCB_AIO_V2.kicad_sch (KiCad schematic)
At the start: 45 parts, among them J1 Conn_01x02_Pin, J2 Conn_01x09_Pin, J3 MPU, J4 STLINK, J5 Conn_01x06_Pin, J6 Conn_01x06_Pin, J7 MPU, Q1 S8550, SW1 SW_Push, SW2 SW_Push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

Commit message: completed PCB_AIO_V2
Parts:
- removed J1: Conn_01x02_Pin, Connector_JST:JST_VH_B2P-VH-B_1x02_P3.96mm_Vertical, symbol Connector:Conn_01x02_Pin
- removed U3: Output 3.3V, Mini560:Mini560_5A, symbol Mini560-5A:Mini560-5A
- added C19: 330uF, Capacitor_Tantalum_SMD:CP_EIA-7343-20_Kemet-V, symbol Device:C_Polarized_Small
- added C20, C21: 10uF, Capacitor_Tantalum_SMD:CP_EIA-3216-10_Kemet-I, symbol Device:C_Polarized_Small
- added J1: EN pin, Connector_PinHeader_2.54mm:PinHeader_1x01_P2.54mm_Vertical, symbol Connector:Conn_01x01_Socket
- added RN2: R_Pack05, Resistor_SMD:R_Array_Convex_5x0603, symbol Device:R_Pack05
- added SW4: SW_DIP_x05, Button_Switch_SMD:SW_DIP_SPSTx05_Slide_KingTek_DSHP05TS_W7.62mm_P1.27mm, symbol Switch:SW_DIP_x05
- added SW5: SW_DPDT_x2, Button_Switch_SMD:SW_SPDT_PCM12, symbol Switch:SW_DPDT_x2
- added U3: AMS1117-3.3, Package_TO_SOT_SMD:SOT-223-3_TabPin2, symbol Regulator_Linear:AMS1117-3.3
- J3, J4: footprint JST254:JST 4 -> Connector_JST:JST_SH_BM04B-SRSS-TB_1x04-1MP_P1.00mm_Vertical
- J5, J6: footprint JST254:JST 6 -> Connector_JST:JST_SH_BM06B-SRSS-TB_1x06-1MP_P1.00mm_Vertical
Connections:
- net RIGHT_MOTOR_02 is gone; now on net RIGHT_MOTOR_O2: J6.6 (Pin_6)
- net +3.3V: now also C21.1, RN2.1 (R1.1), RN2.2 (R2.1), RN2.3 (R3.1), RN2.4 (R4.1), RN2.5 (R5.1), U3.2 (VO); no longer Q1.1 (E)
- net +5V: now also Q1.1 (E), C19.1, C20.1, U3.3 (VI)
- net GND: now also C19.2, C20.2, C21.2, SW5.3 (C), U3.1 (GND)
- net IR_SENSOR_BL: now also U1.25 (PA3); no longer U1.15 (PC0)
- net IR_SENSOR_BR: now also U1.24 (PA2); no longer U1.16 (PC1)
- net IR_SENSOR_FF: now also U1.35 (PB1); no longer U1.30 (PA6)
- net IR_SENSOR_FR: now also U1.15 (PC0); no longer U1.25 (PA3)
- net IR_SENSOR_RL: now also U1.30 (PA6); no longer U1.35 (PB1)
- net IR_SENSOR_RR: now also U1.16 (PC1); no longer U1.24 (PA2)
- net LED_0: now also D1.2 (A), U1.81 (PD0); no longer D4.2 (A), U1.1 (PE2)
- net LED_1: now also D2.2 (A), U1.82 (PD1); no longer D3.2 (A), U1.2 (PE3)
- net LED_2: now also D3.2 (A), U1.83 (PD2); no longer D2.2 (A), U1.3 (PE4)
- net LED_3: now also D4.2 (A), U1.84 (PD3); no longer D1.2 (A), U1.4 (PE5)
- net at D4.1 (K): now also RN1.1 (R1.1); no longer RN1.4 (R4.1)
- net at D1.1 (K): now also RN1.4 (R4.1); no longer RN1.1 (R1.1)
- net at D2.1 (K): now also RN1.3 (R3.1); no longer RN1.2 (R2.1)
- net at D3.1 (K): now also RN1.2 (R2.1); no longer RN1.3 (R3.1)
- net BIT_SW_4: now reaches U1.5 (PE6)
- net BIT_SW_4: now also SW4.6
- net RIGHT_MOTOR_01 renamed RIGHT_MOTOR_O1
- new net: J1.1 (Pin_1), SW5.2 (B)
- new net: RN2.10 (R1.2), SW4.1
- new net: RN2.9 (R2.2), SW4.2
- new net: RN2.8 (R3.2), SW4.3
- new net: RN2.7 (R4.2), SW4.4
- new net: RN2.6 (R5.2), SW4.5
- new net BIT_SW_0: SW4.10, U1.1 (PE2)
- new net BIT_SW_1: SW4.9, U1.2 (PE3)
- new net BIT_SW_2: SW4.8, U1.3 (PE4)
- new net BIT_SW_3: SW4.7, U1.4 (PE5)
Other:
- note added: "BIT SWITCH"
- moved on the sheet: BZ1, D1, D2, D3, D4, Q1, R1, U2

Commit message: SH 1.0 4P -> XH 2.54 4P
Parts:
- J3, J4: footprint Connector_JST:JST_SH_BM04B-SRSS-TB_1x04-1MP_P1.00mm_Vertical -> JST254:JST 4
Changed lines of the file:
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@@
 			)
 		)
-		(property "Footprint" "Connector_JST:JST_SH_BM04B-SRSS-TB_1x04-1MP_P1.00mm_Vertical"
+		(property "Footprint" "JST254:JST 4"
 			(at 494.284 34.544 0)
 			(effects
@@
 			)
 		)
-		(property "Footprint" "Connector_JST:JST_SH_BM04B-SRSS-TB_1x04-1MP_P1.00mm_Vertical"
+		(property "Footprint" "JST254:JST 4"
 			(at 492.506 121.666 0)
 			(effects
